File: UINIO-LCD2.4-ST7789.kicad_pcb (KiCad board)
At the start: 2 copper layers, 69.3 x 48.7 mm, 35 parts, among them CON1 FFC_8Pin_0.5mm, J1 Conn_01x08_Male, Q1 S8050, U1 ME6211C33M5G-N, U2 AMS1117, U3 XC6206P332MR, U4 CON_10Pin

Commit message: Release UINIO-LCD2.4-ST7789 1.0.0.
Parts:
- added ?: LOGO, LOGO, B.Cu at (165.5, 105.5)
- moved U4 0.61 mm to (181.9, 105.6)
Routing:
- net /VDD_3.3V: track 131.3 -> 130.1 mm
- net Net-(R8-Pad2): track 41.5 -> 40.9 mm
- net /SCK: track 41.6 -> 41.0 mm
- net /RES: track 37.9 -> 37.3 mm
- net /MOSI: track 41.8 -> 41.2 mm
- net /DC: track 44.4 -> 43.8 mm
- net /CS: track 47.2 -> 46.6 mm
Other:
- board text added: "UinIO.com"
- board text added: "电子技术博客"

Commit message: Update logo.
Parts:
- removed the ? at (165.5, 105.5)
- added ?: , LOGO, F.Cu at (120.3, 102.1)
- added ?: , LOGO, B.Cu at (148.9, 102.4)
- moved C5 12.2 mm to (151.1, 91.8)
- moved C6 12.2 mm to (127.8, 91.4)
- moved C7 12.2 mm to (153.0, 91.9)
- moved CON1 12.2 mm to (151.0, 102.7)
- moved D4 12.2 mm to (135.3, 106.8)
- moved D5 12.2 mm to (137.9, 106.8)
- moved R1 12.2 mm to (128.3, 101.5)
- moved R2 12.2 mm to (130.6, 101.5)
- moved R3 12.2 mm to (132.9, 101.5)
- moved R4 12.2 mm to (135.3, 101.5)
- moved R6 12.2 mm to (135.7, 91.5)
- moved R7 12.2 mm to (127.8, 88.7)
- moved TP3 12.2 mm to (130.5, 117.3)
- moved TP4 12.2 mm to (133.8, 117.3)
- moved TP5 12.2 mm to (137.1, 117.3)
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Routing:
- net GND: track 27.1 -> 36.3 mm
- net /VDD_3.3V: track 130.1 -> 133.4 mm
- net Net-(CON1-Pad5): track 42.1 -> 41.5 mm
- net Net-(CON1-Pad4): track 43.3 -> 42.8 mm
- net /VDD_5V: track 169.7 -> 169.2 mm
Other:
- board text removed: "UinIO.com"
- board text removed: "电子技术博客"

Commit message: Regerate gerber files.
Parts:
- moved U4 0.54 mm to (169.6, 102.4)
Routing:
- net GND: track 36.3 -> 90.3 mm, vias 2 -> 9
- net /VDD_5V: track 169.2 -> 173.5 mm
- net /VDD_3.3V: track 133.4 -> 131.3 mm
- net Net-(R8-Pad2): track 40.9 -> 40.3 mm
- net /SCK: track 41.0 -> 40.4 mm
- net /RES: track 37.3 -> 36.8 mm
- net /MOSI: track 41.0 -> 40.5 mm
- net /DC: track 43.8 -> 43.2 mm
- net /CS: track 46.6 -> 46.0 mm
